File: eagle/harpscheme.brd (EAGLE design)
At the start: 100 x 80 mm, 67 parts, among them Q1 BC337, Q10 BC327, Q11 BC337, Q12 BC327, Q13 BC337, Q14 BC327, Q15 BC337, Q16 BC327, Q17 BC337, Q18 BC327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

Commit message: eagle - board draft
Parts:
- added J1: (no value), con-amp:10X02MTA
- moved R47 148.8 mm to (74.9, 26.7), turned to 270 degrees
- moved R37 132.8 mm to (59.7, 26.7), turned to 270 degrees
- moved Q13 127.0 mm to (53.3, 34.3)
- moved R43 125.7 mm to (71.1, 26.7), turned to 90 degrees
- moved R27 116.7 mm to (44.5, 26.7), turned to 270 degrees
- moved R42 112.5 mm to (67.3, 26.7), turned to 270 degrees
- moved R33 109.6 mm to (55.9, 26.7), turned to 90 degrees
- moved Q11 106.7 mm to (45.7, 34.3)
- moved R48 106.3 mm to (78.7, 26.7), turned to 90 degrees
- moved R17 100.7 mm to (29.2, 26.7), turned to 270 degrees
- moved R32 96.5 mm to (52.1, 26.7), turned to 270 degrees
- moved R23 93.6 mm to (40.6, 26.7), turned to 90 degrees
- moved R38 90.3 mm to (63.5, 26.7), turned to 90 degrees
- moved Q9 86.4 mm to (38.1, 34.3)
- moved Q3 85.3 mm to (15.2, 34.3)
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Connections:
- net +5V: now also J1.2
- net GND: now also J1.1
Routing:
- net GND: track 47.3 -> 227.8 mm
- net +5V: track 48.0 -> 193.3 mm
- net N$6: track 0.00 -> 35.7 mm
- net N$47: track 0.00 -> 35.4 mm
- net N$12: track 0.00 -> 32.1 mm
- net N$41: track 0.00 -> 31.1 mm
- net N$78: track 5.61 -> 35.7 mm
- net N$66: track 0.00 -> 28.6 mm
- net N$18: track 0.00 -> 28.6 mm
- net N$35: track 0.00 -> 27.5 mm
- net N$71: track 0.00 -> 27.5 mm
- net N$72: track 6.13 -> 32.1 mm
- net N$60: track 0.00 -> 25.0 mm
- net N$24: track 0.00 -> 25.0 mm
- net N$65: track 0.00 -> 22.4 mm
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Other:
- board size 100 x 80 mm -> 105.1 x 61 mm
