File: eagle/harpscheme.sch (EAGLE design)
At the start: 67 parts, among them Q1 BC337, Q10 BC327, Q11 BC337, Q12 BC327, Q13 BC337, Q14 BC327, Q15 BC337, Q16 BC327, Q17 BC337, Q18 BC327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

Commit message: eagle - board draft
Parts:
- added J1: (no value), con-amp:MTA02-100
Connections:
- net +5V: now also J1.2
- net GND: now also J1.1
Changed lines of the file:
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@@
 <part name="GND13" library="supply1" deviceset="GND" device=""/>
 <part name="GND10" library="supply1" deviceset="GND" device=""/>
+<part name="J1" library="con-amp" deviceset="MTA02-100" device=""/>
+<part name="P+2" library="supply1" deviceset="+5V" device=""/>
+<part name="GND14" library="supply1" deviceset="GND" device=""/>
 </parts>
 <sheets>
@@
 <instance part="GND13" gate="1" x="276.86" y="53.34"/>
 <instance part="GND10" gate="1" x="215.9" y="53.34"/>
+<instance part="J1" gate="G$1" x="35.56" y="129.54"/>
+<instance part="P+2" gate="1" x="45.72" y="129.54"/>
+<instance part="GND14" gate="1" x="35.56" y="121.92"/>
 </instances>
 <busses>
@@
 <junction x="45.72" y="93.98"/>
 </segment>
+<segment>
+<pinref part="J1" gate="G$1" pin="2"/>
+<wire x1="38.1" y1="127" x2="38.1" y2="124.46" width="0.1524" layer="91"/>
+<pinref part="P+2" gate="1" pin="+5V"/>
+<wire x1="38.1" y1="124.46" x2="45.72" y2="124.46" width="0.1524" layer="91"/>
+<wire x1="45.72" y1="124.46" x2="45.72" y2="127" width="0.1524" layer="91"/>
+</segment>
 </net>
 <net name="N$4" class="0">
@@
 <wire x1="33.02" y1="55.88" x2="33.02" y2="58.42" width="0.1524" layer="91"/>
 </segment>
-</net>
+<segment>
+<pinref part="J1" gate="G$1" pin="1"/>
+<pinref part="GND14" gate="1" pin="GND"/>
+<wire x1="35.56" y1="127" x2="35.56" y2="124.46" width="0.1524" layer="91"/>
+</segment>
+</net>
